File: Kicad Files/aircond.kicad_sch (KiCad schematic)
At the start: 8 parts, among them SW10 APU BLEED, SW11 PACK1, SW12 PACK2, SW13 EXT_PWR

Commit message: New STL files for APU OVHD element, other coming in the next few weeks
Parts:
- SW10, SW11, SW12, SW13: footprint SFLibrary:G-Switch PS-7054DVB-6PN -> PCM_SFLibrary:G-Switch PS-7054DVB-6PN
Changed lines of the file:
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@@
 (kicad_sch
-	(version 20231120)
+	(version 20250114)
 	(generator "eeschema")
-	(generator_version "8.0")
+	(generator_version "9.0")
 	(paper "A4")
 	(no_connect
@@
 			)
 		)
-		(property "Footprint" "SFLibrary:G-Switch PS-7054DVB-6PN"
+		(property "Footprint" "PCM_SFLibrary:G-Switch PS-7054DVB-6PN"
 			(at 38.1 81.28 0)
 			(effects
@@
 			)
 		)
-		(property "Footprint" "SFLibrary:G-Switch PS-7054DVB-6PN"
+		(property "Footprint" "PCM_SFLibrary:G-Switch PS-7054DVB-6PN"
 			(at 38.1 45.72 0)
 			(effects
@@
 			)
 		)
-		(property "Footprint" "SFLibrary:G-Switch PS-7054DVB-6PN"
+		(property "Footprint" "PCM_SFLibrary:G-Switch PS-7054DVB-6PN"
 			(at 38.1 99.06 0)
 			(effects
@@
 			)
 		)
-		(property "Footprint" "SFLibrary:G-Switch PS-7054DVB-6PN"
+		(property "Footprint" "PCM_SFLibrary:G-Switch PS-7054DVB-6PN"
 			(at 38.1 63.5 0)
 			(effects
