File: Kicad Files/anti_ice_signs.kicad_sch (KiCad schematic)
At the start: 10 parts, among them SW3 ANTI_ICE_WING_SW, SW4 ANTI_ICE_ENG1_SW, SW5 ANTI_ICE_ENG2_SW

Commit message: New STL files for APU OVHD element, other coming in the next few weeks
Parts:
- SW3, SW4, SW5: footprint SFLibrary:G-Switch PS-7054DVB-6PN -> PCM_SFLibrary:G-Switch PS-7054DVB-6PN
Connections:
- net NOSMOKING_OFF: no longer names the net of S10.3
- net NOSMOKING_ON renamed NOSMOKING_SIGN
- net SEATBELTS_OFF: no longer names the net of S9.3
- net SEATBELTS_ON renamed SEATBELTS_SIGN
- no-connect marks 12 -> 14
Changed lines of the file:
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@@
 (kicad_sch
-	(version 20231120)
+	(version 20250114)
 	(generator "eeschema")
-	(generator_version "8.0")
+	(generator_version "9.0")
 	(paper "A4")
 	(no_connect
@@
 	)
 	(no_connect
+		(at 57.15 64.77)
+	)
+	(no_connect
 		(at 99.06 71.12)
 	)
@@
 	(no_connect
 		(at 99.06 73.66)
+	)
+	(no_connect
+		(at 57.15 77.47)
 	)
 	(no_connect
@@
 	(wire
 		(pts
-			(xy 66.04 77.47) (xy 57.15 77.47)
+			(xy 113.03 91.44) (xy 111.76 91.44)
 		)
 		(stroke
@@
 	(wire
 		(pts
-			(xy 113.03 91.44) (xy 111.76 91.44)
+			(xy 66.04 59.69) (xy 57.15 59.69)
 		)
 		(stroke
@@
 	(wire
 		(pts
-			(xy 66.04 59.69) (xy 57.15 59.69)
+			(xy 118.11 57.15) (xy 113.03 57.15)
 		)
 		(stroke
@@
 	(wire
 		(pts
-			(xy 118.11 57.15) (xy 113.03 57.15)
+			(xy 113.03 92.71) (xy 113.03 91.44)
 		)
 		(stroke
@@
 	(wire
 		(pts
-			(xy 113.03 92.71) (xy 113.03 91.44)
+			(xy 118.11 92.71) (xy 113.03 92.71)
 		)
 		(stroke
@@
 	(wire
 		(pts
-			(xy 118.11 92.71) (xy 113.03 92.71)
+			(xy 66.04 87.63) (xy 57.15 87.63)
 		)
 		(stroke
@@
 	(wire
 		(pts
-			(xy 66.04 64.77) (xy 57.15 64.77)
+			(xy 113.03 55.88) (xy 111.76 55.88)
 		)
 		(stroke
@@
 	(wire
 		(pts
-			(xy 66.04 87.63) (xy 57.15 87.63)
+			(xy 114.3 88.9) (xy 111.76 88.9)
 		)
 		(stroke
@@
 	(wire
 		(pts
-			(xy 113.03 55.88) (xy 111.76 55.88)
+			(xy 66.04 72.39) (xy 57.15 72.39)
 		)
 		(stroke
@@
 	(wire
 		(pts
-			(xy 114.3 88.9) (xy 111.76 88.9)
+			(xy 113.03 74.93) (xy 113.03 73.66)
 		)
 		(stroke
@@
 	(wire
 		(pts
-			(xy 66.04 72.39) (xy 57.15 72.39)
+			(xy 118.11 74.93) (xy 113.03 74.93)
 		)
 		(stroke
@@
 	(wire
 		(pts
-			(xy 113.03 74.93) (xy 113.03 73.66)
+			(xy 66.04 92.71) (xy 57.15 92.71)
 		)
 		(stroke
@@
 		)
 	)
-	(wire
-		(pts
-			(xy 118.11 74.93) (xy 113.03 74.93)
-		)
-		(stroke
-			(width 0)
-			(type default)
-		)
-	)
-	(wire
-		(pts
-			(xy 66.04 92.71) (xy 57.15 92.71)
-		)
-		(stroke
-			(width 0)
-			(type default)
-		)
-	)
 	(global_label "ANTI_ICE_ENG1_SW"
 		(shape input)
@@
 		)
 	)
-	(global_label "NOSMOKING_ON"
+	(global_label "NOSMOKING_SIGN"
 		(shape input)
 		(at 66.04 72.39 0)
@@
 		)
 		(property "Intersheetrefs" "${INTERSHEET_REFS}"
-			(at 83.7815 72.39 0)
-			(effects
-				(font
-					(size 1.27 1.27)
-				)
-				(justify left)
-				(hide yes)
-			)
-		)
-	)
-	(global_label "SEATBELTS_ON"
+			(at 85.5353 72.39 0)
+			(effects
+				(font
+					(size 1.27 1.27)
+				)
+				(justify left)
+				(hide yes)
+			)
+		)
+	)
+	(global_label "SEATBELTS_SIGN"
 		(shape input)
 		(at 66.04 59.69 0)
@@
 		)
 		(property "Intersheetrefs" "${INTERSHEET_REFS}"
-			(at 82.6927 59.69 0)
+			(at 84.4465 59.69 0)
 			(effects
 				(font
@@
 		)
 	)
-	(global_label "SEATBELTS_OFF"
+	(global_label "ANTI_ICE_WING_SW"
 		(shape input)
-		(at 66.04 64.77 0)
+		(at 118.11 57.15 0)
 		(fields_autoplaced yes)
 		(effects
@@
 		)
 		(property "Intersheetrefs" "${INTERSHEET_REFS}"
-			(at 83.5394 64.77 0)
-			(effects
-				(font
-					(size 1.27 1.27)
-				)
-				(justify left)
-				(hide yes)
-			)
-		)
-	)
-	(global_label "ANTI_ICE_WING_SW"
+			(at 138.3309 57.15 0)
+			(effects
+				(font
+					(size 1.27 1.27)
+				)
+				(justify left)
+				(hide yes)
+			)
+		)
+	)
+	(global_label "EMERG_ON"
 		(shape input)
-		(at 118.11 57.15 0)
+		(at 66.04 87.63 0)
 		(fields_autoplaced yes)
 		(effects
@@
 		)
 		(property "Intersheetrefs" "${INTERSHEET_REFS}"
-			(at 138.3309 57.15 0)
-			(effects
-				(font
-					(size 1.27 1.27)
-				)
-				(justify left)
-				(hide yes)
-			)
-		)
-	)
-	(global_label "EMERG_ON"
-		(shape input)
-		(at 66.04 87.63 0)
-		(fields_autoplaced yes)
-		(effects
-			(font
-				(size 1.27 1.27)
-			)
-			(justify left)
-		)
-		(property "Intersheetrefs" "${INTERSHEET_REFS}"
 			(at 78.9432 87.63 0)
-			(effects
-				(font
-					(size 1.27 1.27)
-				)
-				(justify left)
-				(hide yes)
-			)
-		)
-	)
-	(global_label "NOSMOKING_OFF"
-		(shape input)
-		(at 66.04 77.47 0)
-		(fields_autoplaced yes)
-		(effects
-			(font
-				(size 1.27 1.27)
-			)
-			(justify left)
-		)
-		(property "Intersheetrefs" "${INTERSHEET_REFS}"
-			(at 84.6282 77.47 0)
 			(effects
 				(font
@@
 			)
 		)
-		(property "Footprint" "SFLibrary:G-Switch PS-7054DVB-6PN"
+		(property "Footprint" "PCM_SFLibrary:G-Switch PS-7054DVB-6PN"
 			(at 106.68 77.47 0)
 			(effects
@@
 			)
 		)
-		(property "Footprint" "SFLibrary:G-Switch PS-7054DVB-6PN"
+		(property "Footprint" "PCM_SFLibrary:G-Switch PS-7054DVB-6PN"
 			(at 106.68 59.69 0)
 			(effects
@@
 			)
 		)
-		(property "Footprint" "SFLibrary:G-Switch PS-7054DVB-6PN"
+		(property "Footprint" "PCM_SFLibrary:G-Switch PS-7054DVB-6PN"
 			(at 106.68 95.25 0)
 			(effects
