File: Kicad Files/apu.kicad_sch (KiCad schematic)
At the start: 6 parts, among them SW1 APU_MASTER_SW, SW2 APU_START_SW

Commit message: New STL files for APU OVHD element, other coming in the next few weeks
Parts:
- SW1, SW2: footprint SFLibrary:G-Switch PS-7054DVB-6PN -> PCM_SFLibrary:G-Switch PS-7054DVB-6PN
Changed lines of the file:
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@@
 (kicad_sch
-	(version 20231120)
+	(version 20250114)
 	(generator "eeschema")
-	(generator_version "8.0")
+	(generator_version "9.0")
 	(paper "A4")
 	(no_connect
@@
 			)
 		)
-		(property "Footprint" "SFLibrary:G-Switch PS-7054DVB-6PN"
+		(property "Footprint" "PCM_SFLibrary:G-Switch PS-7054DVB-6PN"
 			(at 29.21 33.02 0)
 			(effects
@@
 			)
 		)
-		(property "Footprint" "SFLibrary:G-Switch PS-7054DVB-6PN"
+		(property "Footprint" "PCM_SFLibrary:G-Switch PS-7054DVB-6PN"
 			(at 73.66 33.02 0)
 			(effects
