File: Kicad Files/batt.kicad_sch (KiCad schematic)
At the start: 7 parts, among them SW14 OXY_CREW_SUPPLY, SW15 ELEC_BATT_1, SW16 ELEC_BATT_2

Commit message: New STL files for APU OVHD element, other coming in the next few weeks
Parts:
- SW14, SW15, SW16: footprint SFLibrary:G-Switch PS-7054DVB-6PN -> PCM_SFLibrary:G-Switch PS-7054DVB-6PN
Changed lines of the file:
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@@
 (kicad_sch
-	(version 20231120)
+	(version 20250114)
 	(generator "eeschema")
-	(generator_version "8.0")
+	(generator_version "9.0")
 	(paper "A4")
 	(no_connect
@@
 			)
 		)
-		(property "Footprint" "SFLibrary:G-Switch PS-7054DVB-6PN"
+		(property "Footprint" "PCM_SFLibrary:G-Switch PS-7054DVB-6PN"
 			(at 33.02 52.07 0)
 			(effects
@@
 			)
 		)
-		(property "Footprint" "SFLibrary:G-Switch PS-7054DVB-6PN"
+		(property "Footprint" "PCM_SFLibrary:G-Switch PS-7054DVB-6PN"
 			(at 33.02 34.29 0)
 			(effects
@@
 			)
 		)
-		(property "Footprint" "SFLibrary:G-Switch PS-7054DVB-6PN"
+		(property "Footprint" "PCM_SFLibrary:G-Switch PS-7054DVB-6PN"
 			(at 33.02 69.85 0)
 			(effects
