File: Kicad Files/ch340g.kicad_sch (KiCad schematic)
At the start: 30 parts, among them J4 BootLoader, J5 PJ-102A, P1 USB_C_Plug_USB2.0, U2 AMS1117-3.3, U3 CH340G, U4 MIC29302WU

Commit message: Improved pcb design by adding a dip-switch to alter I2C physical address and other small design improvements
Parts:
- XT12MHz1: footprint Crystal:Crystal_SMD_EuroQuartz_MJ-4Pin_5.0x3.2mm_HandSoldering -> Crystal:Crystal_SMD_EuroQuartz_MQ-4Pin_7.0x5.0mm_HandSoldering
Changed lines of the file:
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@@
 			)
 		)
-		(property "Footprint" "Crystal:Crystal_SMD_EuroQuartz_MJ-4Pin_5.0x3.2mm_HandSoldering"
+		(property "Footprint" "Crystal:Crystal_SMD_EuroQuartz_MQ-4Pin_7.0x5.0mm_HandSoldering"
 			(at 133.35 77.47 0)
 			(effects
