File: Kicad Files/dm13a_blue.kicad_sch (KiCad schematic)
At the start: 12 parts, among them U7 DM13A-BLUE

Commit message: VsCode firmware file + changes in the PCB layout
Connections:
- net +5V: no longer RV3.3
- no-connect marks 9 -> 10
Changed lines of the file:
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@@
+	)
+	(no_connect
+		(at 100.33 40.64)
 	)
 	(no_connect
@@
 		(pts
 			(xy 68.58 30.48) (xy 68.58 40.005)
-		)
-		(stroke
-			(width 0)
-			(type default)
-		)
-	)
-	(wire
-		(pts
-			(xy 100.33 34.29) (xy 100.33 40.64)
 		)
 		(stroke
@@
 					(unit 1)
 				)
-			)
-		)
-	)
-	(symbol
-		(lib_id "power:+5V")
-		(at 100.33 34.29 0)
-		(unit 1)
-		(exclude_from_sim no)
-		(in_bom yes)
-		(on_board yes)
-		(dnp no)
-		(fields_autoplaced yes)
-		(property "Reference" "#PWR0167"
-			(at 100.33 38.1 0)
-			(effects
-				(font
-					(size 1.27 1.27)
-				)
-				(hide yes)
-			)
-		)
-		(property "Value" "+5V"
-			(at 100.33 29.21 0)
-			(effects
-				(font
-					(size 1.27 1.27)
-				)
-			)
-		)
-		(property "Footprint" ""
-			(at 100.33 34.29 0)
-			(effects
-				(font
-					(size 1.27 1.27)
-				)
-				(hide yes)
-			)
-		)
-		(property "Datasheet" ""
-			(at 100.33 34.29 0)
-			(effects
-				(font
-					(size 1.27 1.27)
-				)
-				(hide yes)
-			)
-		)
-		(property "Description" "Power symbol creates a global label with name \"+5V\""
-			(at 100.33 34.29 0)
-			(effects
-				(font
-					(size 1.27 1.27)
-				)
-				(hide yes)
-			)
-		)
-		(pin "1"
-		)
-		(instances
-			(project "OverHead_v1"
-				(path "/b62c6a35-e532-4a7b-9786-2edcfc1d7d32/2f7223c5-e8c8-496f-955a-185c9039ce2e"
-					(reference "#PWR0167")
-					(unit 1)
-				)

Commit message: Fixed some issues with the code and path on remote drive
Parts:
- added R52: 56, Resistor_SMD:R_1206_3216Metric_Pad1.30x1.75mm_HandSolder, symbol Device:R
- U7: value DM13A-BLUE -> DM13A-BLUE-0-100
Connections:
- net at C21.2, U7.23 (REXT): now also R52.1; no longer RV3.2
- new net: R52.2, RV3.2
Other:
- moved on the sheet: RV3
Changed lines of the file:
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@@
 	)
 	(no_connect
-		(at 100.33 40.64)
+		(at 113.03 44.45)
 	)
 	(no_connect
@@
 	(wire
 		(pts
-			(xy 95.25 48.26) (xy 95.25 44.45)
-		)
-		(stroke
-			(width 0)
-			(type default)
-		)
-	)
-	(wire
-		(pts
-			(xy 95.25 44.45) (xy 96.52 44.45)
-		)
-		(stroke
-			(width 0)
-			(type default)
-		)
-	)
-	(wire
-		(pts
 			(xy 105.41 81.28) (xy 68.58 81.28)
 		)
@@
 	(wire
 		(pts
+			(xy 104.14 48.26) (xy 109.22 48.26)
+		)
+		(stroke
+			(width 0)
+			(type default)
+		)
+	)
+	(wire
+		(pts
 			(xy 55.88 102.87) (xy 52.07 102.87)
 		)
@@
 	(wire
 		(pts
-			(xy 107.95 48.26) (xy 100.33 48.26)
+			(xy 120.65 52.07) (xy 113.03 52.07)
 		)
 		(stroke
@@
 	(wire
 		(pts
-			(xy 95.25 48.26) (xy 88.9 48.26)
+			(xy 88.9 48.26) (xy 96.52 48.26)
 		)
 		(stroke
@@
 	(symbol
 		(lib_id "power:GND")
-		(at 107.95 48.26 90)
+		(at 120.65 52.07 90)
 		(unit 1)
 		(exclude_from_sim no)
@@
 		(fields_autoplaced yes)
 		(property "Reference" "#PWR0169"
-			(at 114.3 48.26 0)
+			(at 127 52.07 0)
 			(effects
 				(font
@@
 		)
 		(property "Value" "GND"
-			(at 111.76 48.2599 90)
+			(at 124.46 52.0699 90)
 			(effects
 				(font
@@
 		)
 		(property "Footprint" ""
-			(at 107.95 48.26 0)
+			(at 120.65 52.07 0)
 			(effects
 				(font
@@
 		)
 		(property "Datasheet" ""
-			(at 107.95 48.26 0)
+			(at 120.65 52.07 0)
 			(effects
 				(font
@@
 		)
 		(property "Description" "Power symbol creates a global label with name \"GND\" , ground"
-			(at 107.95 48.26 0)
+			(at 120.65 52.07 0)
 			(effects
 				(font
@@
 	)
 	(symbol
+		(lib_id "Device:R")
+		(at 100.33 48.26 90)
+		(unit 1)
+		(exclude_from_sim no)
+		(in_bom yes)
+		(on_board yes)
+		(dnp no)
+		(fields_autoplaced yes)
+		(property "Reference" "R52"
+			(at 100.33 41.91 90)
+			(effects
+				(font
+					(size 1.27 1.27)
+				)
+			)
+		)
+		(property "Value" "56"
+			(at 100.33 44.45 90)
+			(effects
+				(font
+					(size 1.27 1.27)
+				)
+			)
+		)
+		(property "Footprint" "Resistor_SMD:R_1206_3216Metric_Pad1.30x1.75mm_HandSolder"
+			(at 100.33 50.038 90)
+			(effects
+				(font
+					(size 1.27 1.27)
+				)
+				(hide yes)
+			)
+		)
+		(property "Datasheet" "~"
+			(at 100.33 48.26 0)
+			(effects
+				(font
+					(size 1.27 1.27)
+				)
+				(hide yes)
+			)
+		)
+		(property "Description" "Resistor"
+			(at 100.33 48.26 0)
+			(effects
+				(font
+					(size 1.27 1.27)
+				)
+				(hide yes)
+			)
+		)
+		(pin "1"
+		)
+		(pin "2"
+		)
+		(instances
+			(project "OverHead_v1"
+				(path "/b62c6a35-e532-4a7b-9786-2edcfc1d7d32/2f7223c5-e8c8-496f-955a-185c9039ce2e"
+					(reference "R52")
+					(unit 1)
+				)
+			)
+		)
+	)
+	(symbol
 		(lib_id "Device:LED")
 		(at 48.26 125.73 180)
@@
 			)
 		)
-		(property "Value" "DM13A-BLUE"
+		(property "Value" "DM13A-BLUE-0-100"
 			(at 70.7741 40.64 0)
 			(effects
@@
 	(symbol
 		(lib_id "PCM_SL_Devices:potentiometer_3362P")
-		(at 100.33 44.45 90)
+		(at 113.03 48.26 90)
 		(unit 1)
 		(exclude_from_sim no)
@@
 		(fields_autoplaced yes)
 		(property "Reference" "RV3"
-			(at 102.87 43.1799 90)
+			(at 115.57 46.9899 90)
 			(effects
 				(font
@@
 		)
 		(property "Value" "POT_BLUE"
-			(at 102.87 45.7199 90)
+			(at 115.57 49.5299 90)
 			(effects
 				(font
@@
 		)
 		(property "Footprint" "PCM_SL_Footprints:potentiometer_3362P"
-			(at 106.934 44.704 0)
+			(at 119.634 48.514 0)
 			(effects
 				(font
@@
 		)
 		(property "Datasheet" "https://www.bourns.com/data/global/pdfs/3362.pdf"
-			(at 108.966 44.704 0)
+			(at 121.666 48.514 0)
 			(effects
 				(font
@@
 		)
 		(property "Description" "potentiometer_3362P"
-			(at 100.33 44.45 0)
-			(effects
-				(font
+			(at 113.03 48.26 0)
+			(effects
+				(font

Commit message: New STL files for APU OVHD element, other coming in the next few weeks
Parts:
- D109, D126, D129, D130, D131, D132, D133, D4: footprint LED_THT:LED_Rectangular_W3.9mm_H1.8mm_FlatTop -> PCM_LED_THT_AKL:LED_Rectangular_W3.9mm_H1.8mm_FlatTop
Changed lines of the file:
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@@
 (kicad_sch
-	(version 20231120)
+	(version 20250114)
 	(generator "eeschema")
-	(generator_version "8.0")
+	(generator_version "9.0")
 	(paper "A4")
 	(junction
@@
 	(label "LED_GND_CTL_ON"
 		(at 58.42 53.34 180)
-		(fields_autoplaced yes)
 		(effects
 			(font
@@
 	(label "LED_APU_START_ON"
 		(at 80.01 71.12 0)
-		(fields_autoplaced yes)
 		(effects
 			(font
@@
 	(label "LED_ANTI_ICE_ENG1_ON"
 		(at 58.42 60.96 180)
-		(fields_autoplaced yes)
 		(effects
 			(font
@@
 	(label "LED_ANTI_ICE_ENG2_ON"
 		(at 58.42 63.5 180)
-		(fields_autoplaced yes)
 		(effects
 			(font
@@
 	(label "LED_EXT_PWR_ON"
 		(at 58.42 66.04 180)
-		(fields_autoplaced yes)
 		(effects
 			(font
@@
 	(label "LED_EXT_PWR_ON"
 		(at 57.15 171.45 0)
-		(fields_autoplaced yes)
 		(effects
 			(font
@@
 	(label "LED_ANTI_ICE_ENG2_ON"
 		(at 55.88 148.59 0)
-		(fields_autoplaced yes)
 		(effects
 			(font
@@
 	(label "LED_APU_MASTER_ON"
 		(at 55.88 114.3 0)
-		(fields_autoplaced yes)
 		(effects
 			(font
@@
 	(label "LED_ANTI_ICE_WING_ON"
 		(at 57.15 125.73 0)
-		(fields_autoplaced yes)
 		(effects
 			(font
@@
 	(label "LED_APU_START_ON"
 		(at 54.61 160.02 0)
-		(fields_autoplaced yes)
 		(effects
 			(font
@@
 	(label "LED_GND_CTL_ON"
 		(at 55.88 102.87 0)
-		(fields_autoplaced yes)
 		(effects
 			(font
@@
 	(label "LED_ANTI_ICE_WING_ON"
 		(at 58.42 58.42 180)
-		(fields_autoplaced yes)
 		(effects
 			(font
@@
 	(label "LED_APU_BLEED_ON"
 		(at 55.88 182.88 0)
-		(fields_autoplaced yes)
 		(effects
 			(font
@@
 	(label "LED_APU_BLEED_ON"
 		(at 80.01 68.58 0)
-		(fields_autoplaced yes)
 		(effects
 			(font
@@
 	(label "LED_ANTI_ICE_ENG1_ON"
 		(at 55.88 137.16 0)
-		(fields_autoplaced yes)
 		(effects
 			(font
@@
 	(label "LED_APU_MASTER_ON"
 		(at 58.42 55.88 180)
-		(fields_autoplaced yes)
 		(effects
 			(font
@@
 			)
 		)
-		(property "Footprint" "LED_THT:LED_Rectangular_W3.9mm_H1.8mm_FlatTop"
+		(property "Footprint" "PCM_LED_THT_AKL:LED_Rectangular_W3.9mm_H1.8mm_FlatTop"
 			(at 48.26 102.87 0)
 			(effects
@@
 			)
 		)
-		(property "Footprint" "LED_THT:LED_Rectangular_W3.9mm_H1.8mm_FlatTop"
+		(property "Footprint" "PCM_LED_THT_AKL:LED_Rectangular_W3.9mm_H1.8mm_FlatTop"
 			(at 48.26 125.73 0)
 			(effects
@@
 			)
 		)
-		(property "Footprint" "LED_THT:LED_Rectangular_W3.9mm_H1.8mm_FlatTop"
+		(property "Footprint" "PCM_LED_THT_AKL:LED_Rectangular_W3.9mm_H1.8mm_FlatTop"
 			(at 48.26 137.16 0)
 			(effects
@@
 			)
 		)
-		(property "Footprint" "LED_THT:LED_Rectangular_W3.9mm_H1.8mm_FlatTop"
+		(property "Footprint" "PCM_LED_THT_AKL:LED_Rectangular_W3.9mm_H1.8mm_FlatTop"
 			(at 48.26 182.88 0)
 			(effects
@@
 			)
 		)
-		(property "Footprint" "LED_THT:LED_Rectangular_W3.9mm_H1.8mm_FlatTop"
+		(property "Footprint" "PCM_LED_THT_AKL:LED_Rectangular_W3.9mm_H1.8mm_FlatTop"
 			(at 46.99 160.02 0)
 			(effects
@@
 			)
 		)
-		(property "Footprint" "LED_THT:LED_Rectangular_W3.9mm_H1.8mm_FlatTop"
+		(property "Footprint" "PCM_LED_THT_AKL:LED_Rectangular_W3.9mm_H1.8mm_FlatTop"
 			(at 48.26 148.59 0)
 			(effects
@@
 			)
 		)
-		(property "Footprint" "LED_THT:LED_Rectangular_W3.9mm_H1.8mm_FlatTop"
+		(property "Footprint" "PCM_LED_THT_AKL:LED_Rectangular_W3.9mm_H1.8mm_FlatTop"
 			(at 48.26 171.45 0)
 			(effects
@@
 			)
 		)
-		(property "Footprint" "LED_THT:LED_Rectangular_W3.9mm_H1.8mm_FlatTop"
+		(property "Footprint" "PCM_LED_THT_AKL:LED_Rectangular_W3.9mm_H1.8mm_FlatTop"
 			(at 48.26 114.3 0)
 			(effects
