File: Kicad Files/dm13a_white.kicad_sch (KiCad schematic)
At the start: 20 parts, among them U6 DM13A-WHITE

Commit message: VsCode firmware file + changes in the PCB layout
Connections:
- net +5V: no longer RV1.3
- no-connect marks 0 -> 1
Changed lines of the file:
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@@
 		(color 0 0 0 0)
 	)
+	(no_connect
+		(at 97.79 34.29)
+	)
 	(wire
 		(pts
@@
 	(wire
 		(pts
-			(xy 97.79 29.21) (xy 97.79 34.29)
-		)
-		(stroke
-			(width 0)
-			(type default)
-		)
-	)
-	(wire
-		(pts
 			(xy 66.04 74.93) (xy 102.87 74.93)
 		)
@@
 					(unit 1)
 				)
-			)
-		)
-	)
-	(symbol
-		(lib_id "power:+5V")
-		(at 97.79 29.21 0)
-		(unit 1)
-		(exclude_from_sim no)
-		(in_bom yes)
-		(on_board yes)
-		(dnp no)
-		(fields_autoplaced yes)
-		(property "Reference" "#PWR0212"
-			(at 97.79 33.02 0)
-			(effects
-				(font
-					(size 1.27 1.27)
-				)
-				(hide yes)
-			)
-		)
-		(property "Value" "+5V"
-			(at 97.79 24.13 0)
-			(effects
-				(font
-					(size 1.27 1.27)
-				)
-			)
-		)
-		(property "Footprint" ""
-			(at 97.79 29.21 0)
-			(effects
-				(font
-					(size 1.27 1.27)
-				)
-				(hide yes)
-			)
-		)
-		(property "Datasheet" ""
-			(at 97.79 29.21 0)
-			(effects
-				(font
-					(size 1.27 1.27)
-				)
-				(hide yes)
-			)
-		)
-		(property "Description" "Power symbol creates a global label with name \"+5V\""
-			(at 97.79 29.21 0)
-			(effects
-				(font
-					(size 1.27 1.27)
-				)
-				(hide yes)
-			)
-		)
-		(pin "1"
-		)
-		(instances
-			(project "OverHead_v1"
-				(path "/b62c6a35-e532-4a7b-9786-2edcfc1d7d32/2f1b9fe8-b81e-49ed-9171-b387b6e501b8"
-					(reference "#PWR0212")
-					(unit 1)
-				)

Commit message: Fixed some issues with the code and path on remote drive
Parts:
- added R51: 56, Resistor_SMD:R_1206_3216Metric_Pad1.30x1.75mm_HandSolder, symbol Device:R
- U6: value DM13A-WHITE -> DM13A-WHITE-0-100
Connections:
- net at C17.2, U6.23 (REXT): now also R51.1; no longer RV1.2
- new net: R51.2, RV1.2
Other:
- moved on the sheet: RV1
Changed lines of the file:
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@@
 	)
 	(no_connect
-		(at 97.79 34.29)
+		(at 106.68 38.1)
 	)
 	(wire
@@
 	(wire
 		(pts
-			(xy 92.71 41.91) (xy 92.71 38.1)
-		)
-		(stroke
-			(width 0)
-			(type default)
-		)
-	)
-	(wire
-		(pts
 			(xy 123.19 165.1) (xy 119.38 165.1)
 		)
@@
 	(wire
 		(pts
-			(xy 105.41 41.91) (xy 97.79 41.91)
+			(xy 114.3 45.72) (xy 106.68 45.72)
 		)
 		(stroke
@@
 	(wire
 		(pts
-			(xy 92.71 38.1) (xy 93.98 38.1)
-		)
-		(stroke
-			(width 0)
-			(type default)
-		)
-	)
-	(wire
-		(pts
 			(xy 77.47 41.91) (xy 86.36 41.91)
 		)
@@
 	(wire
 		(pts
+			(xy 99.06 41.91) (xy 102.87 41.91)
+		)
+		(stroke
+			(width 0)
+			(type default)
+		)
+	)
+	(wire
+		(pts
 			(xy 123.19 142.24) (xy 119.38 142.24)
 		)
@@
 	(wire
 		(pts
-			(xy 92.71 41.91) (xy 86.36 41.91)
+			(xy 86.36 41.91) (xy 91.44 41.91)
 		)
 		(stroke
@@
 	(symbol
 		(lib_id "PCM_SL_Devices:potentiometer_3362P")
-		(at 97.79 38.1 90)
+		(at 106.68 41.91 90)
 		(unit 1)
 		(exclude_from_sim no)
@@
 		(fields_autoplaced yes)
 		(property "Reference" "RV1"
-			(at 100.33 36.8299 90)
+			(at 109.22 40.6399 90)
 			(effects
 				(font
@@
 		)
 		(property "Value" "POT_WHITE"
-			(at 100.33 39.3699 90)
+			(at 109.22 43.1799 90)
 			(effects
 				(font
@@
 		)
 		(property "Footprint" "PCM_SL_Footprints:potentiometer_3362P"
-			(at 104.394 38.354 0)
+			(at 113.284 42.164 0)
 			(effects
 				(font
@@
 		)
 		(property "Datasheet" "https://www.bourns.com/data/global/pdfs/3362.pdf"
-			(at 106.426 38.354 0)
+			(at 115.316 42.164 0)
 			(effects
 				(font
@@
 		)
 		(property "Description" "potentiometer_3362P"
-			(at 97.79 38.1 0)
+			(at 106.68 41.91 0)
 			(effects
 				(font
@@
 	)
 	(symbol
+		(lib_id "Device:R")
+		(at 95.25 41.91 90)
+		(unit 1)
+		(exclude_from_sim no)
+		(in_bom yes)
+		(on_board yes)
+		(dnp no)
+		(fields_autoplaced yes)
+		(property "Reference" "R51"
+			(at 95.25 35.56 90)
+			(effects
+				(font
+					(size 1.27 1.27)
+				)
+			)
+		)
+		(property "Value" "56"
+			(at 95.25 38.1 90)
+			(effects
+				(font
+					(size 1.27 1.27)
+				)
+			)
+		)
+		(property "Footprint" "Resistor_SMD:R_1206_3216Metric_Pad1.30x1.75mm_HandSolder"
+			(at 95.25 43.688 90)
+			(effects
+				(font
+					(size 1.27 1.27)
+				)
+				(hide yes)
+			)
+		)
+		(property "Datasheet" "~"
+			(at 95.25 41.91 0)
+			(effects
+				(font
+					(size 1.27 1.27)
+				)
+				(hide yes)
+			)
+		)
+		(property "Description" "Resistor"
+			(at 95.25 41.91 0)
+			(effects
+				(font
+					(size 1.27 1.27)
+				)
+				(hide yes)
+			)
+		)
+		(pin "1"
+		)
+		(pin "2"
+		)
+		(instances
+			(project "OverHead_v1"
+				(path "/b62c6a35-e532-4a7b-9786-2edcfc1d7d32/2f1b9fe8-b81e-49ed-9171-b387b6e501b8"
+					(reference "R51")
+					(unit 1)
+				)
+			)
+		)
+	)
+	(symbol
 		(lib_id "Device:LED")
 		(at 115.57 176.53 180)
@@
 			)
 		)
-		(property "Value" "DM13A-WHITE"
+		(property "Value" "DM13A-WHITE-0-100"
 			(at 68.2341 34.29 0)
 			(effects
@@
 	(symbol
 		(lib_id "power:GND")
-		(at 105.41 41.91 90)
+		(at 114.3 45.72 90)
 		(unit 1)
 		(exclude_from_sim no)
@@
 		(fields_autoplaced yes)
 		(property "Reference" "#PWR0211"
-			(at 111.76 41.91 0)
+			(at 120.65 45.72 0)
 			(effects
 				(font
@@
 		)
 		(property "Value" "GND"
-			(at 109.22 41.9099 90)
+			(at 118.11 45.7199 90)
 			(effects
 				(font
@@
 		)
 		(property "Footprint" ""
-			(at 105.41 41.91 0)
+			(at 114.3 45.72 0)
 			(effects
 				(font
@@
 		)
 		(property "Datasheet" ""
-			(at 105.41 41.91 0)
+			(at 114.3 45.72 0)
 			(effects
 				(font
@@
 		)
 		(property "Description" "Power symbol creates a global label with name \"GND\" , ground"
-			(at 105.41 41.91 0)
+			(at 114.3 45.72 0)
 			(effects
 				(font

Commit message: New STL files for APU OVHD element, other coming in the next few weeks
Parts:
- D103, D106, D107, D120, D121, D122, D123, D124, D125, D127, D76, D78, D79, D80, D90, D92: footprint LED_THT:LED_Rectangular_W3.9mm_H1.8mm_FlatTop -> PCM_LED_THT_AKL:LED_Rectangular_W3.9mm_H1.8mm_FlatTop
Changed lines of the file:
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@@
 (kicad_sch
-	(version 20231120)
+	(version 20250114)
 	(generator "eeschema")
-	(generator_version "8.0")
+	(generator_version "9.0")
 	(paper "A4")
 	(junction
@@
 	(label "LED_RT_TK_PUMP_2_OFF"
 		(at 123.19 176.53 0)
-		(fields_autoplaced yes)
 		(effects
 			(font
@@
 	(label "LED_GPWS_TERR_OFF"
 		(at 80.01 119.38 0)
-		(fields_autoplaced yes)
 		(effects
 			(font
@@
 	(label "LED_PACK2_OFF"
 		(at 166.37 119.38 0)
-		(fields_autoplaced yes)
 		(effects
 			(font
@@
 	(label "LED_XFEED_ON"
 		(at 123.19 142.24 0)
-		(fields_autoplaced yes)
 		(effects
 			(font
@@
 	(label "LED_RT_TK_PUMP_2_OFF"
 		(at 77.47 62.23 0)
-		(fields_autoplaced yes)
 		(effects
 			(font
@@
 	(label "LED_L_XFER_OFF"
 		(at 123.19 130.81 0)
-		(fields_autoplaced yes)
 		(effects
 			(font
@@
 	(label "LED_ELEC_BATT_2_OFF"
 		(at 77.47 49.53 0)
-		(fields_autoplaced yes)
 		(effects
 			(font
@@
 	(label "LED_LT_TK_PUMP_2_OFF"
 		(at 55.88 62.23 180)
-		(fields_autoplaced yes)
 		(effects
 			(font
@@
 	(label "LED_OXY_CREW_SUPPLY_OFF"
 		(at 55.88 57.15 180)
-		(fields_autoplaced yes)
 		(effects
 			(font
@@
 	(label "LED_L_XFER_OFF"
 		(at 55.88 64.77 180)
-		(fields_autoplaced yes)
 		(effects
 			(font
@@
 	(label "LED_GPWS_SYS_OFF"
 		(at 55.88 49.53 180)
-		(fields_autoplaced yes)
 		(effects
 			(font
@@
 	(label "LED_PACK1_OFF"
 		(at 166.37 107.95 0)
-		(fields_autoplaced yes)
 		(effects
 			(font
@@
 	(label "LED_GPWS_TERR_OFF"
 		(at 55.88 46.99 180)
-		(fields_autoplaced yes)
 		(effects
 			(font
@@
 	(label "LED_R_XFER_OFF"
 		(at 77.47 57.15 0)
-		(fields_autoplaced yes)
 		(effects
 			(font
@@
 	(label "LED_ELEC_BATT_1_OFF"
 		(at 77.47 46.99 0)
-		(fields_autoplaced yes)
 		(effects
 			(font
@@
 	(label "LED_LT_TK_PUMP_1_OFF"
 		(at 123.19 107.95 0)
-		(fields_autoplaced yes)
 		(effects
 			(font
@@
 	(label "LED_FLAPS3_OFF"
 		(at 40.64 179.07 0)
-		(fields_autoplaced yes)
 		(effects
 			(font
@@
 	(label "LED_RT_TK_PUMP_1_OFF"
 		(at 77.47 59.69 0)
-		(fields_autoplaced yes)
 		(effects
 			(font
@@
 	(label "LED_ELEC_BATT_2_OFF"
 		(at 81.28 143.51 0)
-		(fields_autoplaced yes)
 		(effects
 			(font
@@
 	(label "LED_LT_TK_PUMP_2_OFF"
 		(at 123.19 119.38 0)
-		(fields_autoplaced yes)
 		(effects
 			(font
@@
 	(label "LED_PACK2_OFF"
 		(at 77.47 54.61 0)
-		(fields_autoplaced yes)
 		(effects
 			(font
@@
 	(label "LED_PACK1_OFF"
 		(at 77.47 64.77 0)
-		(fields_autoplaced yes)
 		(effects
 			(font
@@
 	(label "LED_ELEC_BATT_1_OFF"
 		(at 81.28 130.81 0)
-		(fields_autoplaced yes)
 		(effects
 			(font
@@
 	(label "LED_GS_OFF"
 		(at 40.64 167.64 0)
-		(fields_autoplaced yes)
 		(effects
 			(font
@@
 	(label "LED_OXY_CREW_SUPPLY_OFF"
 		(at 80.01 156.21 0)
-		(fields_autoplaced yes)
 		(effects
 			(font
@@
 	(label "LED_RT_TK_PUMP_1_OFF"
 		(at 123.19 165.1 0)
-		(fields_autoplaced yes)
 		(effects
 			(font
@@
 	(label "LED_XFEED_ON"
 		(at 77.47 52.07 0)
-		(fields_autoplaced yes)
 		(effects
 			(font
@@
 	(label "LED_FLAPS3_OFF"
 		(at 55.88 54.61 180)
-		(fields_autoplaced yes)
 		(effects
 			(font
@@
 	(label "LED_LT_TK_PUMP_1_OFF"
 		(at 55.88 59.69 180)
-		(fields_autoplaced yes)
 		(effects
 			(font
@@
 	(label "LED_GPWS_SYS_OFF"
 		(at 40.64 156.21 0)
-		(fields_autoplaced yes)
 		(effects
 			(font
@@
 	(label "LED_R_XFER_OFF"
 		(at 123.19 153.67 0)
-		(fields_autoplaced yes)
 		(effects
 			(font
@@
 	(label "LED_GS_OFF"
 		(at 55.88 52.07 180)
-		(fields_autoplaced yes)
 		(effects
 			(font
@@
 			)
 		)
-		(property "Footprint" "LED_THT:LED_Rectangular_W3.9mm_H1.8mm_FlatTop"
+		(property "Footprint" "PCM_LED_THT_AKL:LED_Rectangular_W3.9mm_H1.8mm_FlatTop"
 			(at 72.39 143.51 0)
 			(effects
@@
 			)
 		)
-		(property "Footprint" "LED_THT:LED_Rectangular_W3.9mm_H1.8mm_FlatTop"
+		(property "Footprint" "PCM_LED_THT_AKL:LED_Rectangular_W3.9mm_H1.8mm_FlatTop"
 			(at 158.75 107.95 0)
 			(effects
@@
 			)
 		)
-		(property "Footprint" "LED_THT:LED_Rectangular_W3.9mm_H1.8mm_FlatTop"
+		(property "Footprint" "PCM_LED_THT_AKL:LED_Rectangular_W3.9mm_H1.8mm_FlatTop"
 			(at 72.39 130.81 0)
 			(effects
@@
 			)
 		)
-		(property "Footprint" "LED_THT:LED_Rectangular_W3.9mm_H1.8mm_FlatTop"
+		(property "Footprint" "PCM_LED_THT_AKL:LED_Rectangular_W3.9mm_H1.8mm_FlatTop"
 			(at 115.57 165.1 0)
 			(effects
@@
 			)
 		)
-		(property "Footprint" "LED_THT:LED_Rectangular_W3.9mm_H1.8mm_FlatTop"
+		(property "Footprint" "PCM_LED_THT_AKL:LED_Rectangular_W3.9mm_H1.8mm_FlatTop"
 			(at 115.57 130.81 0)
 			(effects
@@
 			)
 		)
-		(property "Footprint" "LED_THT:LED_Rectangular_W3.9mm_H1.8mm_FlatTop"
+		(property "Footprint" "PCM_LED_THT_AKL:LED_Rectangular_W3.9mm_H1.8mm_FlatTop"
 			(at 33.02 156.21 0)
 			(effects
@@
 			)
 		)
-		(property "Footprint" "LED_THT:LED_Rectangular_W3.9mm_H1.8mm_FlatTop"
+		(property "Footprint" "PCM_LED_THT_AKL:LED_Rectangular_W3.9mm_H1.8mm_FlatTop"
 			(at 115.57 153.67 0)
 			(effects
@@
 			)
 		)
-		(property "Footprint" "LED_THT:LED_Rectangular_W3.9mm_H1.8mm_FlatTop"
+		(property "Footprint" "PCM_LED_THT_AKL:LED_Rectangular_W3.9mm_H1.8mm_FlatTop"
 			(at 115.57 107.95 0)
 			(effects
@@
 			)
 		)
-		(property "Footprint" "LED_THT:LED_Rectangular_W3.9mm_H1.8mm_FlatTop"
+		(property "Footprint" "PCM_LED_THT_AKL:LED_Rectangular_W3.9mm_H1.8mm_FlatTop"
 			(at 115.57 176.53 0)
 			(effects
@@
 			)
 		)
-		(property "Footprint" "LED_THT:LED_Rectangular_W3.9mm_H1.8mm_FlatTop"
+		(property "Footprint" "PCM_LED_THT_AKL:LED_Rectangular_W3.9mm_H1.8mm_FlatTop"
 			(at 33.02 179.07 0)
 			(effects
@@
 			)
 		)
-		(property "Footprint" "LED_THT:LED_Rectangular_W3.9mm_H1.8mm_FlatTop"
+		(property "Footprint" "PCM_LED_THT_AKL:LED_Rectangular_W3.9mm_H1.8mm_FlatTop"
 			(at 33.02 167.64 0)
 			(effects
@@
 			)
 		)
-		(property "Footprint" "LED_THT:LED_Rectangular_W3.9mm_H1.8mm_FlatTop"
+		(property "Footprint" "PCM_LED_THT_AKL:LED_Rectangular_W3.9mm_H1.8mm_FlatTop"
 			(at 115.57 142.24 0)
 			(effects
@@
 			)
 		)
-		(property "Footprint" "LED_THT:LED_Rectangular_W3.9mm_H1.8mm_FlatTop"
+		(property "Footprint" "PCM_LED_THT_AKL:LED_Rectangular_W3.9mm_H1.8mm_FlatTop"
 			(at 72.39 119.38 0)
 			(effects
@@
 			)
 		)
-		(property "Footprint" "LED_THT:LED_Rectangular_W3.9mm_H1.8mm_FlatTop"
+		(property "Footprint" "PCM_LED_THT_AKL:LED_Rectangular_W3.9mm_H1.8mm_FlatTop"
 			(at 158.75 119.38 0)
 			(effects
@@
 			)
 		)
-		(property "Footprint" "LED_THT:LED_Rectangular_W3.9mm_H1.8mm_FlatTop"
+		(property "Footprint" "PCM_LED_THT_AKL:LED_Rectangular_W3.9mm_H1.8mm_FlatTop"
 			(at 115.57 119.38 0)
 			(effects
@@
 			)
 		)
-		(property "Footprint" "LED_THT:LED_Rectangular_W3.9mm_H1.8mm_FlatTop"
+		(property "Footprint" "PCM_LED_THT_AKL:LED_Rectangular_W3.9mm_H1.8mm_FlatTop"
 			(at 72.39 156.21 0)
 			(effects
