File: Kicad Files/fuel.kicad_sch (KiCad schematic)
At the start: 12 parts, among them SW17 LT_TK_PUMP_1, SW18 LT_TK_PUMP_2, SW19 L_XFER, SW20 X_FEED, SW21 R_XFER, SW22 RT_TK_PUMP_1, SW23 RT_TK_PUMP_2

Commit message: New STL files for APU OVHD element, other coming in the next few weeks
Parts:
- SW17, SW18, SW19, SW20, SW21, SW22, SW23: footprint SFLibrary:G-Switch PS-7054DVB-6PN -> PCM_SFLibrary:G-Switch PS-7054DVB-6PN
Connections:
- net L_XFER_SW renamed CTR_TK_PUMP_1_SW
- net R_XFER_SW renamed CTR_TK_PUMP_2_SW
Changed lines of the file:
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@@
 (kicad_sch
-	(version 20231120)
+	(version 20250114)
 	(generator "eeschema")
-	(generator_version "8.0")
+	(generator_version "9.0")
 	(paper "A4")
 	(no_connect
@@
 		)
 	)
-	(global_label "L_XFER_SW"
+	(global_label "CTR_TK_PUMP_1_SW"
 		(shape input)
 		(at 33.02 62.23 0)
@@
 		)
 		(property "Intersheetrefs" "${INTERSHEET_REFS}"
-			(at 46.3465 62.23 0)
+			(at 54.8131 62.23 0)
 			(effects
 				(font
@@
 		)
 	)
-	(global_label "R_XFER_SW"
+	(global_label "CTR_TK_PUMP_2_SW"
 		(shape input)
 		(at 33.02 97.79 0)
@@
 		)
 		(property "Intersheetrefs" "${INTERSHEET_REFS}"
-			(at 46.5884 97.79 0)
+			(at 54.8131 97.79 0)
 			(effects
 				(font
@@
 			)
 		)
-		(property "Footprint" "SFLibrary:G-Switch PS-7054DVB-6PN"
+		(property "Footprint" "PCM_SFLibrary:G-Switch PS-7054DVB-6PN"
 			(at 27.94 101.6 0)
 			(effects
@@
 			)
 		)
-		(property "Footprint" "SFLibrary:G-Switch PS-7054DVB-6PN"
+		(property "Footprint" "PCM_SFLibrary:G-Switch PS-7054DVB-6PN"
 			(at 27.94 83.82 0)
 			(effects
@@
 			)
 		)
-		(property "Footprint" "SFLibrary:G-Switch PS-7054DVB-6PN"
+		(property "Footprint" "PCM_SFLibrary:G-Switch PS-7054DVB-6PN"
 			(at 27.94 119.38 0)
 			(effects
@@
 			)
 		)
-		(property "Footprint" "SFLibrary:G-Switch PS-7054DVB-6PN"
+		(property "Footprint" "PCM_SFLibrary:G-Switch PS-7054DVB-6PN"
 			(at 27.94 48.26 0)
 			(effects
@@
 			)
 		)
-		(property "Footprint" "SFLibrary:G-Switch PS-7054DVB-6PN"
+		(property "Footprint" "PCM_SFLibrary:G-Switch PS-7054DVB-6PN"
 			(at 27.94 30.48 0)
 			(effects
@@
 			)
 		)
-		(property "Footprint" "SFLibrary:G-Switch PS-7054DVB-6PN"
+		(property "Footprint" "PCM_SFLibrary:G-Switch PS-7054DVB-6PN"
 			(at 27.94 66.04 0)
 			(effects
@@
 			)
 		)
-		(property "Footprint" "SFLibrary:G-Switch PS-7054DVB-6PN"
+		(property "Footprint" "PCM_SFLibrary:G-Switch PS-7054DVB-6PN"
 			(at 27.94 137.16 0)
 			(effects
