File: Kicad Files/gwps.kicad_sch (KiCad schematic)
At the start: 8 parts, among them SW6 TERR, SW7 SYS, SW8 G/S MODE, SW9 LDG FLAPS 3

Commit message: New STL files for APU OVHD element, other coming in the next few weeks
Parts:
- SW6, SW7, SW8, SW9: footprint SFLibrary:G-Switch PS-7054DVB-6PN -> PCM_SFLibrary:G-Switch PS-7054DVB-6PN
Changed lines of the file:
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@@
 (kicad_sch
-	(version 20231120)
+	(version 20250114)
 	(generator "eeschema")
-	(generator_version "8.0")
+	(generator_version "9.0")
 	(paper "A4")
 	(no_connect
@@
 			)
 		)
-		(property "Footprint" "SFLibrary:G-Switch PS-7054DVB-6PN"
+		(property "Footprint" "PCM_SFLibrary:G-Switch PS-7054DVB-6PN"
 			(at 43.18 81.28 0)
 			(effects
@@
 			)
 		)
-		(property "Footprint" "SFLibrary:G-Switch PS-7054DVB-6PN"
+		(property "Footprint" "PCM_SFLibrary:G-Switch PS-7054DVB-6PN"
 			(at 43.18 99.06 0)
 			(effects
@@
 			)
 		)
-		(property "Footprint" "SFLibrary:G-Switch PS-7054DVB-6PN"
+		(property "Footprint" "PCM_SFLibrary:G-Switch PS-7054DVB-6PN"
 			(at 43.18 45.72 0)
 			(effects
@@
 			)
 		)
-		(property "Footprint" "SFLibrary:G-Switch PS-7054DVB-6PN"
+		(property "Footprint" "PCM_SFLibrary:G-Switch PS-7054DVB-6PN"
 			(at 43.18 63.5 0)
 			(effects
