File: Kicad Files/OverHead_v1.kicad_pcb (KiCad board)
At the start: 4 copper layers, 313 x 206 mm, 416 parts, among them J1 BATT_1_OLED, J2 BATT_2_OLED, J3 ADIRS_OLED, J4 BootLoader, J5 PJ-102A, P1 USB_C_Plug_USB2.0, SW1 APU_MASTER_SW, SW10 APU BLEED, SW11 PACK1, SW12 PACK2, SW13 EXT_PWR, SW14 OXY_CREW_SUPPLY, SW15 ELEC_BATT_1, SW16 ELEC_BATT_2, SW17 LT_TK_PUMP_1, SW18 LT_TK_PUMP_2, SW19 L_XFER, SW2 APU_START_SW, SW20 X_FEED, SW21 R_XFER, SW22 RT_TK_PUMP_1, SW23 RT_TK_PUMP_2, SW24 GND_CTL, SW25 ADR_1, SW26 ADR_2, SW27 ADR_3, SW28 SW_DIP_x03, SW3 ANTI_ICE_WING_SW, SW4 ANTI_ICE_ENG1_SW, SW5 ANTI_ICE_ENG2_SW, SW6 TERR, SW7 SYS, SW8 G/S MODE, SW9 LDG FLAPS 3, U1 ATMega2560, U2 AMS1117-3.3, U3 CH340G, U4 MIC29302WU, U5 DM13A-GREEN-0-100, U6 DM13A-WHITE-0-100, U7 DM13A-BLUE-0-100, U8 DM13A-ORANGE-0-100

Commit message: Put back the v1 project as it was sent to JLCPCB, with the rotaries fixed
The board in the panel was ordered on 3 March 2025. The Gerbers uploaded to
JLCPCB for that order are byte-identical to production/OverHead_v1.zip,
exported that evening at 22:08. KiCad backed the project up at 22:06 and
at 22:26, with the same copper in both. This restores the 22:26 snapshot:
the board, the schematic sheets and the project files.

Its one flaw is in the file, not in the copper. On 22 February the three
ADIRS rotaries used SimPanel:Rotary_SW_8x1_SF, the footprint made for the
switches actually bought, whose pins sit one position round. By 3 March an
update from the schematic had put the library Rotary_SW_8x1 back under
the same tracks. The copper still reached the right physical pins, but the
file showed nine nets unconnected. The three footprints are taken back from
the 22 February board, with the same position, symbol link and nets. The
schematic now names _SF too, so the next update cannot undo it.

Checked on the result: the DRC finds 0 unconnected items. Following the
copper rather than the net names, each of the 49 buttons in the .mfmc
reaches exactly one switch contact, and each of the 44 annunciator outputs
reaches exactly one LED. The two "shorts" the DRC reports are copper the
schematic never drew: NO SMOKING's contact 3 on D5 and SEAT BELTS'
contact 3 on D18. The .mfmc reads NO SMOKING on D5, so the copper is what
works.

Co-Authored-By: Claude Opus 5.5 <noreply@anthropic.com>
Parts:
- SW25, SW26, SW27: footprint SimPanel:Rotary_SW_8x1 -> SimPanel:Rotary_SW_8x1_SF
Connections:
- net SEATBELTS_SIGN renamed SEATBELTS_ON
- S10 pad 1: NOSMOKING_SIGN -> NOSMOKING_ON
- S10 pad 3: unconnected-(S10-Pad3) -> NOSMOKING_OFF
- S9 pad 3: unconnected-(S9-Pad3) -> SEATBELTS_OFF
- U1 pad 5: NOSMOKING_SIGN -> unconnected-(U1-PE3-Pad5)
- U1 pad 50: unconnected-(U1-PD7-Pad50) -> NOSMOKING_ON
Routing:
- net unconnected-(U1-PD7-Pad50): track 197.6 -> 0.00 mm, vias 1 -> 0
- net NOSMOKING_ON: track 0.00 -> 197.6 mm, vias 0 -> 1
- net ADR_1_OFF: track 0.00 -> 181.3 mm, vias 0 -> 1
- net NOSMOKING_OFF: track 0.00 -> 163.6 mm, vias 0 -> 1
- net SEATBELTS_OFF: track 0.00 -> 160.5 mm, vias 0 -> 1
- net ADR_1_NAV: track 0.00 -> 160.3 mm, vias 0 -> 2
- net ADR_1_ATT: track 0.00 -> 156.2 mm, vias 0 -> 2
- net ADR_2_OFF: track 0.00 -> 140.0 mm, vias 0 -> 1
- net ADR_2_NAV: track 0.00 -> 137.1 mm, vias 0 -> 1
- net ADR_2_ATT: track 0.00 -> 122.5 mm, vias 0 -> 1
- net ADR_3_OFF: track 0.00 -> 103.0 mm, vias 0 -> 2
- net ADR_3_NAV: track 0.00 -> 97.0 mm, vias 0 -> 2
- net ADR_3_ATT: track 0.00 -> 95.5 mm, vias 0 -> 2
