File: Kicad Files/adirs.kicad_sch (KiCad schematic)
At the start: 8 parts, among them SW24 GND_CTL, SW25 ADR_1, SW26 ADR_2, SW27 ADR_3

Commit message: Put back the v1 project as it was sent to JLCPCB, with the rotaries fixed
The board in the panel was ordered on 3 March 2025. The Gerbers uploaded to
JLCPCB for that order are byte-identical to production/OverHead_v1.zip,
exported that evening at 22:08. KiCad backed the project up at 22:06 and
at 22:26, with the same copper in both. This restores the 22:26 snapshot:
the board, the schematic sheets and the project files.

Its one flaw is in the file, not in the copper. On 22 February the three
ADIRS rotaries used SimPanel:Rotary_SW_8x1_SF, the footprint made for the
switches actually bought, whose pins sit one position round. By 3 March an
update from the schematic had put the library Rotary_SW_8x1 back under
the same tracks. The copper still reached the right physical pins, but the
file showed nine nets unconnected. The three footprints are taken back from
the 22 February board, with the same position, symbol link and nets. The
schematic now names _SF too, so the next update cannot undo it.

Checked on the result: the DRC finds 0 unconnected items. Following the
copper rather than the net names, each of the 49 buttons in the .mfmc
reaches exactly one switch contact, and each of the 44 annunciator outputs
reaches exactly one LED. The two "shorts" the DRC reports are copper the
schematic never drew: NO SMOKING's contact 3 on D5 and SEAT BELTS'
contact 3 on D18. The .mfmc reads NO SMOKING on D5, so the copper is what
works.

Co-Authored-By: Claude Opus 5.5 <noreply@anthropic.com>
Parts:
- SW25, SW26, SW27: footprint SimPanel:Rotary_SW_8x1 -> SimPanel:Rotary_SW_8x1_SF
Changed lines of the file:
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@@
 			)
 		)
-		(property "Footprint" "SimPanel:Rotary_SW_8x1"
+		(property "Footprint" "SimPanel:Rotary_SW_8x1_SF"
 			(at 46.99 121.92 0)
 			(effects
@@
 			)
 		)
-		(property "Footprint" "SimPanel:Rotary_SW_8x1"
+		(property "Footprint" "SimPanel:Rotary_SW_8x1_SF"
 			(at 46.99 87.63 0)
 			(effects
@@
 			)
 		)
-		(property "Footprint" "SimPanel:Rotary_SW_8x1"
+		(property "Footprint" "SimPanel:Rotary_SW_8x1_SF"
 			(at 46.99 54.61 0)
 			(effects
