File: Section_AIRCOND/Section_AIRCOND.kicad_sch (KiCad schematic)
At the start: 46 parts, among them J1 AIRCOND ribbon, J2 Backlight, SW1 AIRCOND APU BLEED, SW2 AIRCOND PACK 1, SW3 AIRCOND PACK 2, SW4 AIRCOND EXT PWR

Commit message: Single-LED backlight strings on 330 ohm, not 470
A pair of backlight LEDs on 150 ohm runs at 17 mA (Stefano's figure). The
470 ohm came from an estimated 11 mA per string, which was wrong. For the
same 17 mA a single LED needs V / (2 I) + 75 ohm = 330 ohm. Changed on APU
(R3), GPWS (R5), AIR COND (R7, the v1 R76) and EXT LT (R16); the document's
backlight currents now use 17 mA, ~1.1 A in all. The four boards rebuilt
and rerouted: ERC 0, DRC 0, nothing unconnected, no parity issues.

Co-Authored-By: Claude Opus 5.5 <noreply@anthropic.com>
Parts:
- R7: value 470 -> 330
