File: Section_APU/Section_APU.kicad_sch (KiCad schematic)
At the start: 24 parts, among them J1 APU ribbon, J2 Backlight, SW1 APU MASTER SW, SW2 APU START

Commit message: Single-LED backlight strings on 330 ohm, not 470
A pair of backlight LEDs on 150 ohm runs at 17 mA (Stefano's figure). The
470 ohm came from an estimated 11 mA per string, which was wrong. For the
same 17 mA a single LED needs V / (2 I) + 75 ohm = 330 ohm. Changed on APU
(R3), GPWS (R5), AIR COND (R7, the v1 R76) and EXT LT (R16); the document's
backlight currents now use 17 mA, ~1.1 A in all. The four boards rebuilt
and rerouted: ERC 0, DRC 0, nothing unconnected, no parity issues.

Co-Authored-By: Claude Opus 5.5 <noreply@anthropic.com>
Parts:
- R3: value 470 -> 330
