File: Section_GPWS/Section_GPWS.kicad_pcb (KiCad board)
At the start: 2 copper layers, 159.5 x 39 mm, 38 parts, among them J1 GPWS ribbon, J2 Backlight, SW1 GPWS TERR, SW2 GPWS SYS, SW3 GPWS G/S MODE, SW4 GPWS LDG FLAPS 3

Commit message: Single-LED backlight strings on 330 ohm, not 470
A pair of backlight LEDs on 150 ohm runs at 17 mA (Stefano's figure). The
470 ohm came from an estimated 11 mA per string, which was wrong. For the
same 17 mA a single LED needs V / (2 I) + 75 ohm = 330 ohm. Changed on APU
(R3), GPWS (R5), AIR COND (R7, the v1 R76) and EXT LT (R16); the document's
backlight currents now use 17 mA, ~1.1 A in all. The four boards rebuilt
and rerouted: ERC 0, DRC 0, nothing unconnected, no parity issues.

Co-Authored-By: Claude Opus 5.5 <noreply@anthropic.com>
Parts:
- R5: value 470 -> 330
