File: Section_EXTLT/Section_EXTLT.kicad_pcb (KiCad board)
At the start: 2 copper layers, 159.5 x 79.5 mm, 61 parts, among them J1 EXTLT ribbon, J2 Backlight, SW1 EXTLT STROBE, SW2 EXTLT BEACON, SW3 EXTLT WING, SW4 EXTLT NAV & LOGO, SW5 EXTLT RWY TURN, SW6 EXTLT LDG LIGHT L, SW7 EXTLT LDG LIGHT R, SW8 EXTLT NOSE LIGHT

Commit message: Single-LED backlight strings on 330 ohm, not 470
A pair of backlight LEDs on 150 ohm runs at 17 mA (Stefano's figure). The
470 ohm came from an estimated 11 mA per string, which was wrong. For the
same 17 mA a single LED needs V / (2 I) + 75 ohm = 330 ohm. Changed on APU
(R3), GPWS (R5), AIR COND (R7, the v1 R76) and EXT LT (R16); the document's
backlight currents now use 17 mA, ~1.1 A in all. The four boards rebuilt
and rerouted: ERC 0, DRC 0, nothing unconnected, no parity issues.

Co-Authored-By: Claude Opus 5.5 <noreply@anthropic.com>
Parts:
- R16: value 470 -> 330

Commit message: Mainboard schematic: 3.5 mm backlight terminals, IRLIZ44N lying flat
The eight backlight terminals become Phoenix PT 1,5/2-3,5 (22-24 AWG, 1.1 A
in all), so they fit along one edge of the 137 x 89 mm mainboard; the 9 V
input keeps its 5.08 mm terminal. The IRLIZ44N lies flat (TO-220F
horizontal): 1.1 A needs no heatsink, and it stays well below the section
boards. F101's note now says ~1.1 A (63 strings at 17 mA). The netlist
changes only in those nine footprints. The TLC5927 footprint drops a
duplicated pin-1 asterisk. Net classes set for the mainboard layout.

EXT LT: J2 moves next to J1, over the low part of the mainboard.

Co-Authored-By: Claude Opus 5.5 <noreply@anthropic.com>
Parts:
- moved J2 29.7 mm to (199.0, 105.0)
Routing:
- net +9V_BL: track 359.8 -> 379.8 mm, vias 5 -> 6
- net WING_LIGHTS: track 81.1 -> 62.3 mm, vias 0 -> 1
- net BL_RET: track 461.5 -> 446.0 mm, vias 2 -> 5
- net STROBE: track 126.2 -> 138.2 mm
- net R_LDG_LIGHT_ON: track 58.4 -> 70.3 mm, vias 2 -> 0
- net BL2_MID: track 26.3 -> 14.4 mm
- net NOSELIGHT_OFF: track 45.0 -> 33.3 mm, vias 0 -> 2
- net L_LDG_LIGHT_RETR: track 104.2 -> 92.8 mm
- net BL9_MID: track 13.2 -> 21.3 mm
- net R_LDG_LIGHT_RETR: track 60.2 -> 67.7 mm, vias 2 -> 1
- net BL14_R: track 20.4 -> 27.3 mm, vias 0 -> 2
- net GND: track 269.9 -> 263.1 mm
- net L_LDG_LIGHT_ON: track 101.3 -> 107.1 mm
- net BL12_MID: track 14.8 -> 20.5 mm
- net BL6_MID: track 26.7 -> 21.1 mm
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