File: Section_EXTLT/Section_EXTLT.kicad_sch (KiCad schematic)
At the start: 61 parts, among them J1 EXTLT ribbon, J2 Backlight, SW1 EXTLT STROBE, SW2 EXTLT BEACON, SW3 EXTLT WING, SW4 EXTLT NAV & LOGO, SW5 EXTLT RWY TURN, SW6 EXTLT LDG LIGHT L, SW7 EXTLT LDG LIGHT R, SW8 EXTLT NOSE LIGHT

Commit message: Single-LED backlight strings on 330 ohm, not 470
A pair of backlight LEDs on 150 ohm runs at 17 mA (Stefano's figure). The
470 ohm came from an estimated 11 mA per string, which was wrong. For the
same 17 mA a single LED needs V / (2 I) + 75 ohm = 330 ohm. Changed on APU
(R3), GPWS (R5), AIR COND (R7, the v1 R76) and EXT LT (R16); the document's
backlight currents now use 17 mA, ~1.1 A in all. The four boards rebuilt
and rerouted: ERC 0, DRC 0, nothing unconnected, no parity issues.

Co-Authored-By: Claude Opus 5.5 <noreply@anthropic.com>
Parts:
- R16: value 470 -> 330
