File: Mainboard/OVHD_Mainboard.kicad_pcb (KiCad board)
At the start: 2 copper layers, 137 x 89 mm, 130 parts, among them J101 9V IN, J201 BootLoader, J601 ADIRS backlight, J602 FUEL backlight, J603 ELEC backlight, J604 GPWS backlight, J605 AIRCOND backlight, J606 EXTLT backlight, J607 APU backlight, J608 SIGNS backlight, J701 ADIRS ribbon, J702 FUEL ribbon, J703 ELEC ribbon, J704 GPWS ribbon, J705 AIRCOND ribbon, J706 EXTLT ribbon, J707 APU ribbon, J708 SIGNS ribbon, P201 USB_B, Q501 AO3401A, Q502 BS170, Q503 AO3401A, Q504 BS170, Q601 IRLIZ44N, SW401 I2C ADDR, U101 MIC29302WU, U201 CH340G, U202 AMS1117-3.3, U203 TPS2115A, U301 ATmega2560-16AU, U401 PCA9548APW, U501 TLC5927IDWR, U502 TLC5927IDWR, U503 TLC5927IDWR, U504 TLC5927IDWR, Y201 12MHz, Y301 16MHz

Commit message: Take the R-EXT capacitors off the mainboard: they were the fault
On the v1 board each TLC5927 has 100 nF from R-EXT to GND, which the
datasheet's application circuit does not have. With 1 kOhm on R-EXT a
chip dropped all its outputs to under 1 mA as soon as two or three were
on together, and kept them there until a power cycle. Supply, R-EXT, OE
and temperature read the same before and after, and the fault showed
with both firmwares and both Connector command formats. With C17 removed,
U6 held all 16 outputs on while U7, still with its capacitor, failed in
the same test.

C511-C514 go from the v2 schematic and PCB, with the R-EXT stubs that led
to them. ERC, DRC and schematic parity stay at zero. The design document,
the readmes and the mainboard renders follow, and the main readme tells
v1 builders to remove C17, C19, C21 and C23.

Co-Authored-By: Claude Opus 5.5 <noreply@anthropic.com>
Parts:
- removed C511, C512, C513, C514: 100nF, Capacitor_SMD:C_1206_3216Metric_Pad1.33x1.80mm_HandSolder
Routing:
- net U503_REXT: track 24.5 -> 11.4 mm
- net U502_REXT: track 17.5 -> 10.5 mm
- net U504_REXT: track 17.6 -> 10.8 mm

Commit message: Bleed +5V_TLC with 4.7 kOhm, so the TLC5927 reset is sure
When D46 switches the chips off, their supply had only its 10.4 uF and
the chips' own current to fall by. R527, 4.7 kOhm to GND beside C505,
gives it a 49 ms time constant: after the firmware's 300 ms about 10 mV
are left. It costs about 1 mA while the chips are on.

ERC, DRC and schematic parity stay at zero. The renders, the part counts
and the firmware comments follow.

Co-Authored-By: Claude Opus 5.5 <noreply@anthropic.com>
Parts:
- added R527: 4.7K, Resistor_SMD:R_1206_3216Metric_Pad1.30x1.75mm_HandSolder, B.Cu at (98.5, 208.0)
Routing:
- net +5V_TLC: track 138.1 -> 140.6 mm
Changed lines of the file:
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@@
 	(footprint "Resistor_SMD:R_1206_3216Metric_Pad1.30x1.75mm_HandSolder"
 		(layer "B.Cu")
+		(at 98.5 208)
+		(descr "Resistor SMD 1206 (3216 Metric), square (rectangular) end terminal, IPC-7351 nominal with elongated pad for handsoldering. (Body size source: IPC-SM-782 page 72, https://www.pcb-3d.com/wordpress/wp-content/uploads/ipc-sm-782a_amendment_1_and_2.pdf)")
+		(tags "resistor handsolder")
+		(property "Reference" "R527"
+			(at 0 1.83 180)
+			(layer "B.Fab")
+			(effects
+				(font
+					(size 1 1)
+					(thickness 0.15)
+				)
+				(justify mirror)
+			)
+		)
+		(property "Value" "4.7K"
+			(at 0 -1.83 180)
+			(layer "B.Fab")
+			(effects
+				(font
+					(size 1 1)
+					(thickness 0.15)
+				)
+				(justify mirror)
+			)
+		)
+		(property "Datasheet" ""
+			(at 0 0 180)
+			(layer "B.Fab")
+			(hide yes)
+			(effects
+				(font
+					(size 1.27 1.27)
+				)
+				(justify mirror)
+			)
+		)
+		(property "Description" "Bleeds +5V_TLC when D46 switches the chips off, so the reset is sure: 4.7k x 10.4 uF = 49 ms."
+			(at 0 0 180)
+			(layer "B.Fab")
+			(hide yes)
+			(effects
+				(font
+					(size 1.27 1.27)
+				)
+				(justify mirror)
+			)
+		)
+		(property "KiLib_Generator" "SMD_2terminal_chip_molded"
+			(at 0 0 180)
+			(layer "B.SilkS")
+			(hide yes)
+			(effects
+				(font
+					(size 1 1)
+					(thickness 0.15)
+				)
+				(justify mirror)
+			)
+		)
+		(attr smd)
+		(duplicate_pad_numbers_are_jumpers no)
+		(fp_line
+			(start -0.727064 -0.91)
+			(end 0.727064 -0.91)
+			(stroke
+				(width 0.12)
+				(type solid)
+			)
+			(layer "B.SilkS")
+		)
+		(fp_line
+			(start -0.727064 0.91)
+			(end 0.727064 0.91)
+			(stroke
+				(width 0.12)
+				(type solid)
+			)
+			(layer "B.SilkS")
+		)
+		(fp_rect
+			(start -2.45 1.13)
+			(end 2.45 -1.13)
+			(stroke
+				(width 0.05)
+				(type solid)
+			)
+			(fill no)
+			(layer "B.CrtYd")
+		)
+		(fp_rect
+			(start -1.6 0.8)
+			(end 1.6 -0.8)
+			(stroke
+				(width 0.1)
+				(type solid)
+			)
+			(fill no)
+			(layer "B.Fab")
+		)
+		(fp_text user "4.7K"
+			(at 0 2.32 0)
+			(layer "B.SilkS")
+			(effects
+				(font
+					(size 0.8 0.8)
+					(thickness 0.15)
+				)
+				(justify mirror)
+			)
+		)
+		(fp_text user "${REFERENCE}"
+			(at 0 0 180)
+			(layer "B.Fab")
+			(effects
+				(font
+					(size 0.8 0.8)
+					(thickness 0.12)
+				)
+				(justify mirror)
+			)
+		)
+		(pad "1" smd roundrect
+			(at -1.55 0)
+			(size 1.3 1.75)
+			(layers "B.Cu" "B.Mask" "B.Paste")
+			(roundrect_rratio 0.192308)
+			(net "+5V_TLC")
+		)
+		(pad "2" smd roundrect
+			(at 1.55 0)
+			(size 1.3 1.75)
+			(layers "B.Cu" "B.Mask" "B.Paste")
+			(roundrect_rratio 0.192308)
+			(net "GND")
+		)
+		(embedded_fonts no)
+		(model "${KICAD10_3DMODEL_DIR}/Resistor_SMD.3dshapes/R_1206_3216Metric.step"
+			(offset
+				(xyz 0 0 0)
+			)
+			(scale
+				(xyz 1 1 1)
+			)
+			(rotate
+				(xyz 0 0 0)
+			)
+		)
+	)
+	(footprint "Resistor_SMD:R_1206_3216Metric_Pad1.30x1.75mm_HandSolder"
+		(layer "B.Cu")
 		(at 127.5 179)
 		(descr "Resistor SMD 1206 (3216 Metric), square (rectangular) end terminal, IPC-7351 nominal with elongated pad for handsoldering. (Body size source: IPC-SM-782 page 72, https://www.pcb-3d.com/wordpress/wp-content/uploads/ipc-sm-782a_amendment_1_and_2.pdf)")
@@
 		(width 0.25)
 		(layer "B.Cu")
+		(net "+5V_TLC")
+	)
+	(segment
+		(start 96.95 208)
+		(end 96.94 205.49)
+		(width 0.25)
+		(layer "B.Cu")
