File: Mainboard/annunciators.kicad_sch (KiCad schematic)
At the start: 38 parts, among them Q501 AO3401A, Q502 BS170, Q503 AO3401A, Q504 BS170, U501 TLC5927IDWR, U502 TLC5927IDWR, U503 TLC5927IDWR, U504 TLC5927IDWR

Commit message: Lay the mainboard schematic out so that nothing overlaps
Reference and value now sit outside each symbol (above and below, or beside
it for parts whose pins leave up and down), turned horizontal on rotated
parts. GND on a sideways pin is a label instead of a power symbol that
crowded the neighbouring pins. The annunciator sheet keeps its four TLC5927
in two wider columns, their R-EXT and capacitors in a row underneath, the
series resistors horizontal on the right and both supply switches along the
bottom, all inside the frame. The connector sheet has wider columns.

Layout only: the netlist is identical to the previous commit (126 parts,
230 nets, same values, footprints and fields), and ERC is still clean.

Co-Authored-By: Claude Opus 5.5 <noreply@anthropic.com>
Other:
- note added: "Anode rail switch (D45) and TLC5927 supply switch (D46)"
- note added: "Bulk capacitors"
- note added: "Series resistors on CLK / LE / SDI"

Commit message: Take the R-EXT capacitors off the mainboard: they were the fault
On the v1 board each TLC5927 has 100 nF from R-EXT to GND, which the
datasheet's application circuit does not have. With 1 kOhm on R-EXT a
chip dropped all its outputs to under 1 mA as soon as two or three were
on together, and kept them there until a power cycle. Supply, R-EXT, OE
and temperature read the same before and after, and the fault showed
with both firmwares and both Connector command formats. With C17 removed,
U6 held all 16 outputs on while U7, still with its capacitor, failed in
the same test.

C511-C514 go from the v2 schematic and PCB, with the R-EXT stubs that led
to them. ERC, DRC and schematic parity stay at zero. The design document,
the readmes and the mainboard renders follow, and the main readme tells
v1 builders to remove C17, C19, C21 and C23.

Co-Authored-By: Claude Opus 5.5 <noreply@anthropic.com>
Parts:
- removed C511, C512, C513, C514: 100nF, Capacitor_SMD:C_1206_3216Metric_Pad1.33x1.80mm_HandSolder, symbol Device:C

Commit message: Bleed +5V_TLC with 4.7 kOhm, so the TLC5927 reset is sure
When D46 switches the chips off, their supply had only its 10.4 uF and
the chips' own current to fall by. R527, 4.7 kOhm to GND beside C505,
gives it a 49 ms time constant: after the firmware's 300 ms about 10 mV
are left. It costs about 1 mA while the chips are on.

ERC, DRC and schematic parity stay at zero. The renders, the part counts
and the firmware comments follow.

Co-Authored-By: Claude Opus 5.5 <noreply@anthropic.com>
Parts:
- added R527: 4.7K, Resistor_SMD:R_1206_3216Metric_Pad1.30x1.75mm_HandSolder, symbol Device:R
Connections:
- net +5V_TLC: now also R527.1
- net GND: now also R527.2
Changed lines of the file:
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@@
+	)
+	(symbol
+		(lib_id "Device:R")
+		(at 345.44 160.02 0)
+		(unit 1)
+		(body_style 1)
+		(exclude_from_sim no)
+		(in_bom yes)
+		(on_board yes)
+		(in_pos_files yes)
+		(dnp no)
+		(property "Reference" "R527"
+			(at 348.742 158.75 0)
+			(show_name no)
+			(do_not_autoplace no)
+			(effects
+				(font
+					(size 1.27 1.27)
+				)
+				(justify left)
+			)
+		)
+		(property "Value" "4.7K"
+			(at 348.742 161.29 0)
+			(show_name no)
+			(do_not_autoplace no)
+			(effects
+				(font
+					(size 1.27 1.27)
+				)
+				(justify left)
+			)
+		)
+		(property "Footprint" "Resistor_SMD:R_1206_3216Metric_Pad1.30x1.75mm_HandSolder"
+			(at 345.44 160.02 0)
+			(hide yes)
+			(show_name no)
+			(do_not_autoplace no)
+			(effects
+				(font
+					(size 1.27 1.27)
+				)
+			)
+		)
+		(property "Datasheet" ""
+			(at 345.44 160.02 0)
+			(hide yes)
+			(show_name no)
+			(do_not_autoplace no)
+			(effects
+				(font
+					(size 1.27 1.27)
+				)
+			)
+		)
+		(property "Description" "Bleeds +5V_TLC when D46 switches the chips off, so the reset is sure: 4.7k x 10.4 uF = 49 ms."
+			(at 345.44 160.02 0)
+			(show_name no)
+			(do_not_autoplace no)
+			(effects
+				(font
+					(size 1.27 1.27)
+				)
+			)
+		)
+		(pin "1"
+		)
+		(pin "2"
+		)
+		(instances
+			(project "OVHD_Mainboard"
+				(path "/3267b3f3-6c63-480a-8354-1757ed0a4fd3/150a38c8-5b68-4222-97ef-c099286f02a1"
+					(reference "R527")
+					(unit 1)
+				)
+			)
+		)
+	)
+	(symbol
+		(lib_id "power:GND")
+		(at 345.44 163.83 0)
+		(unit 1)
+		(body_style 1)
+		(exclude_from_sim no)
+		(in_bom yes)
+		(on_board yes)
+		(in_pos_files yes)
+		(dnp no)
+		(property "Reference" "#PWR02a1100"
+			(at 345.44 163.83 0)
+			(hide yes)
+			(show_name no)
+			(do_not_autoplace no)
+			(effects
+				(font
+					(size 1.27 1.27)
+				)
+			)
+		)
+		(property "Value" "GND"
+			(at 345.44 167.64 0)
+			(show_name no)
+			(do_not_autoplace no)
+			(effects
+				(font
+					(size 1.27 1.27)
+				)
+			)
+		)
+		(property "Footprint" ""
+			(at 345.44 163.83 0)
+			(hide yes)
+			(show_name no)
+			(do_not_autoplace no)
+			(effects
+				(font
+					(size 1.27 1.27)
+				)
+			)
+		)
+		(property "Datasheet" ""
+			(at 345.44 163.83 0)
+			(hide yes)
+			(show_name no)
+			(do_not_autoplace no)
+			(effects
+				(font
+					(size 1.27 1.27)
+				)
+			)
+		)
+		(property "Description" ""
+			(at 345.44 163.83 0)
+			(show_name no)
+			(do_not_autoplace no)
+			(effects
+				(font
+					(size 1.27 1.27)
+				)
+			)
+		)
+		(pin "1"
+		)
+		(instances
+			(project "OVHD_Mainboard"
+				(path "/3267b3f3-6c63-480a-8354-1757ed0a4fd3/150a38c8-5b68-4222-97ef-c099286f02a1"
+					(reference "#PWR02a1100")
+					(unit 1)
+				)
+			)
+		)
+	)
+	(global_label "+5V_TLC"
+		(shape passive)
+		(at 345.44 156.21 90)
+		(fields_autoplaced yes)
+		(effects
+			(font
+				(size 1.27 1.27)
+			)
+			(justify left)
+		)
+		(property "Intersheetrefs" "${INTERSHEET_REFS}"
+			(at 345.44 156.21 0)
+			(hide yes)
+			(show_name no)
+			(do_not_autoplace no)
+			(effects
+				(font
+					(size 1.27 1.27)
+				)
+			)
+		)
 	)
 	(symbol
